File: design/non-inverting-buck-boost/board-v1/NIBB.sch (EAGLE design)
At the start: 13 parts, among them Q1 IRLZ44Z, Q2 IRLZ44Z

Commit message: replaced fets
Parts:
- IC1, IC2: value ZXGD3006E6 -> (none)
- Q1, Q2: value IRLZ44Z -> (none); device transistor-power:IRLZ44Z -> felippe:IRF640
- renumbered U$1 to IC1, U$2 to IC2
Changed lines of the file:
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@@
 <part name="D1" library="diode" deviceset="MUR820" device=""/>
 <part name="D2" library="diode" deviceset="MUR820" device=""/>
-<part name="Q1" library="transistor-power" deviceset="IRLZ44Z" device=""/>
 <part name="L1" library="inductors" deviceset="RKE16" device=""/>
-<part name="Q2" library="transistor-power" deviceset="IRLZ44Z" device=""/>
 <part name="VLINE" library="con-molex" deviceset="22-23-2021" device="" value=""/>
-<part name="U$1" library="felippe" deviceset="ZXGD3006E6" device=""/>
-<part name="U$2" library="felippe" deviceset="ZXGD3006E6" device=""/>
 <part name="15V" library="con-molex" deviceset="22-23-2021" device="" value=""/>
 <part name="IN" library="con-molex" deviceset="22-23-2021" device="" value=""/>
@@
 <part name="C1" library="capacitor" deviceset="CAPP-U" device="F"/>
 <part name="OUT" library="con-molex" deviceset="22-23-2021" device="" value=""/>
+<part name="IC1" library="felippe" deviceset="ZXGD3006E6" device=""/>
+<part name="IC2" library="felippe" deviceset="ZXGD3006E6" device=""/>
+<part name="Q1" library="felippe" deviceset="IRF640" device=""/>
+<part name="Q2" library="felippe" deviceset="IRF640" device=""/>
 </parts>
 <sheets>
@@
 <instance part="D1" gate="1" x="25.4" y="48.26" rot="R90"/>
 <instance part="D2" gate="1" x="66.04" y="63.5"/>
-<instance part="Q1" gate="G$1" x="17.78" y="60.96" rot="R90"/>
 <instance part="L1" gate="1" x="40.64" y="63.5"/>
-<instance part="Q2" gate="G$1" x="53.34" y="45.72"/>
 <instance part="VLINE" gate="-1" x="-24.13" y="63.5" rot="R180"/>
 <instance part="VLINE" gate="-2" x="-24.13" y="35.56" rot="R180"/>
-<instance part="U$1" gate="G$1" x="12.7" y="50.8"/>
-<instance part="U$2" gate="G$1" x="40.64" y="45.72"/>
 <instance part="15V" gate="-1" x="-22.86" y="58.42" smashed="yes" rot="R180">
 <attribute name="NAME" x="-25.4" y="59.182" size="1.524" layer="95" rot="R180"/>
@@
 </instance>
 <instance part="OUT" gate="-2" x="93.98" y="35.56"/>
+<instance part="IC1" gate="G$1" x="12.7" y="50.8"/>
+<instance part="IC2" gate="G$1" x="40.64" y="45.72"/>
+<instance part="Q1" gate="G$1" x="17.78" y="60.96" rot="R90"/>
+<instance part="Q2" gate="G$1" x="53.34" y="45.72"/>
 </instances>
 <busses>
@@
 <pinref part="D2" gate="1" pin="A"/>
 <wire x1="48.26" y1="63.5" x2="55.88" y2="63.5" width="0.1524" layer="91"/>
-<pinref part="Q2" gate="G$1" pin="D"/>
 <wire x1="55.88" y1="63.5" x2="63.5" y2="63.5" width="0.1524" layer="91"/>
 <wire x1="55.88" y1="50.8" x2="55.88" y2="63.5" width="0.1524" layer="91"/>
 <junction x="55.88" y="63.5"/>
+<pinref part="Q2" gate="G$1" pin="D"/>
 </segment>
 </net>
 <net name="N$4" class="0">
 <segment>
-<pinref part="Q2" gate="G$1" pin="S"/>
 <wire x1="55.88" y1="40.64" x2="55.88" y2="35.56" width="0.1524" layer="91"/>
 <pinref part="VLINE" gate="-2" pin="S"/>
@@
 <wire x1="91.44" y1="35.56" x2="81.28" y2="35.56" width="0.1524" layer="91"/>
 <junction x="81.28" y="35.56"/>
+<pinref part="Q2" gate="G$1" pin="S"/>
 </segment>
 </net>
 <net name="N$3" class="0">
 <segment>
-<pinref part="Q1" gate="G$1" pin="D"/>
 <pinref part="VLINE" gate="-1" pin="S"/>
 <wire x1="-21.59" y1="63.5" x2="12.7" y2="63.5" width="0.1524" layer="91"/>
+<pinref part="Q1" gate="G$1" pin="D"/>
 </segment>
 </net>
 <net name="N$5" class="0">
 <segment>
-<pinref part="U$1" gate="G$1" pin="SOURCE"/>
 <wire x1="17.78" y1="53.34" x2="20.32" y2="53.34" width="0.1524" layer="91"/>
-<pinref part="Q1" gate="G$1" pin="G"/>
 <wire x1="20.32" y1="53.34" x2="20.32" y2="58.42" width="0.1524" layer="91"/>
-<pinref part="U$1" gate="G$1" pin="SINK"/>
 <wire x1="17.78" y1="48.26" x2="20.32" y2="48.26" width="0.1524" layer="91"/>
 <wire x1="20.32" y1="48.26" x2="20.32" y2="53.34" width="0.1524" layer="91"/>
+<pinref part="IC1" gate="G$1" pin="SOURCE"/>
+<pinref part="IC1" gate="G$1" pin="SINK"/>
+<pinref part="Q1" gate="G$1" pin="G"/>
 </segment>
 </net>
 <net name="N$6" class="0">
 <segment>
-<pinref part="U$2" gate="G$1" pin="SOURCE"/>
 <wire x1="48.26" y1="48.26" x2="45.72" y2="48.26" width="0.1524" layer="91"/>
 <wire x1="48.26" y1="43.18" x2="48.26" y2="48.26" width="0.1524" layer="91"/>
-<pinref part="U$2" gate="G$1" pin="SINK"/>
 <wire x1="45.72" y1="43.18" x2="48.26" y2="43.18" width="0.1524" layer="91"/>
+<wire x1="48.26" y1="43.18" x2="50.8" y2="43.18" width="0.1524" layer="91"/>
+<pinref part="IC2" gate="G$1" pin="SOURCE"/>
+<pinref part="IC2" gate="G$1" pin="SINK"/>
 <pinref part="Q2" gate="G$1" pin="G"/>
-<wire x1="48.26" y1="43.18" x2="50.8" y2="43.18" width="0.1524" layer="91"/>
 </segment>
 </net>
@@
 </segment>
 <segment>
-<pinref part="U$1" gate="G$1" pin="VCC"/>
 <wire x1="7.62" y1="53.34" x2="5.08" y2="53.34" width="0.1524" layer="91"/>
 <label x="7.62" y="55.88" size="1.778" layer="95" rot="R180"/>
-</segment>
-<segment>
-<pinref part="U$2" gate="G$1" pin="VCC"/>
+<pinref part="IC1" gate="G$1" pin="VCC"/>
+</segment>
+<segment>
 <wire x1="35.56" y1="48.26" x2="33.02" y2="48.26" width="0.1524" layer="91"/>
 <label x="35.56" y="50.8" size="1.778" layer="95" rot="R180"/>
+<pinref part="IC2" gate="G$1" pin="VCC"/>
 </segment>
 </net>
@@
 </segment>
 <segment>
-<pinref part="U$1" gate="G$1" pin="VEE"/>
 <wire x1="7.62" y1="48.26" x2="5.08" y2="48.26" width="0.1524" layer="91"/>
 <label x="7.62" y="50.8" size="1.778" layer="95" rot="R180"/>
-</segment>
-<segment>
-<pinref part="U$2" gate="G$1" pin="VEE"/>
+<pinref part="IC1" gate="G$1" pin="VEE"/>
+</segment>
+<segment>
 <wire x1="35.56" y1="43.18" x2="33.02" y2="43.18" width="0.1524" layer="91"/>
 <label x="35.56" y="45.72" size="1.778" layer="95" rot="R180"/>
+<pinref part="IC2" gate="G$1" pin="VEE"/>
 </segment>
 </net>
@@
 </segment>
 <segment>
-<pinref part="U$1" gate="G$1" pin="IN"/>
 <wire x1="7.62" y1="50.8" x2="5.08" y2="50.8" width="0.1524" layer="91"/>
 <label x="7.62" y="53.34" size="1.778" layer="95" rot="R180"/>
+<pinref part="IC1" gate="G$1" pin="IN"/>
 </segment>
 </net>
@@
 </segment>
 <segment>
-<pinref part="U$2" gate="G$1" pin="IN"/>
 <wire x1="35.56" y1="45.72" x2="33.02" y2="45.72" width="0.1524" layer="91"/>
 <label x="35.56" y="48.26" size="1.778" layer="95" rot="R180"/>
+<pinref part="IC2" gate="G$1" pin="IN"/>
 </segment>
 </net>
@@
 <net name="N$1" class="0">
 <segment>
-<pinref part="Q1" gate="G$1" pin="S"/>
 <pinref part="L1" gate="1" pin="1"/>
 <wire x1="22.86" y1="63.5" x2="25.4" y2="63.5" width="0.1524" layer="91"/>
@@
 <wire x1="25.4" y1="50.8" x2="25.4" y2="63.5" width="0.1524" layer="91"/>
 <junction x="25.4" y="63.5"/>
-</segment>
-</net>
+<pinref part="Q1" gate="G$1" pin="S"/>
+</segment>
+</net>
